File: astronomer.kicad_sch (KiCad schematic)
At the start: 46 parts, among them J1 6P6C, SW1 SW_Push_45deg, SW10 SW_Push_45deg, SW11 SW_Push_45deg, SW12 SW_Push_45deg, SW13 SW_Push_45deg, SW14 SW_Push_45deg, SW15 SW_Push_45deg, SW16 SW_Push_45deg, SW17 SW_Push_45deg, SW18 SW_Push_45deg, SW19 SW_Push_45deg, SW2 SW_Push_45deg, SW20 SW_Push_45deg, SW21 SW_Push_45deg, SW22 SW_Push_45deg, SW3 SW_Push_45deg, SW4 SW_Push_45deg, SW5 SW_Push_45deg, SW6 SW_Push_45deg, SW7 SW_Push_45deg, SW8 SW_Push_45deg, SW9 SW_Push_45deg

Commit message: lights sch
Parts:
- added C1, C2, C3, C4, C5, C6, C7, C8: C_Small, symbol Device:C_Small
- added D23, D24, D25, D26, D27, D28, D29, D30, D31, D32, D33, D34, D35, D36, D37, D38, D39, D40, D41, D42, D43, D44, D45, D46: SK6812MINI, LED_SMD:LED_SK6812MINI_PLCC4_3.5x3.5mm_P1.75mm, symbol LED:SK6812MINI
Connections:
- net +5V: now also C1.1, C2.1, C3.1, C4.1, C5.1, C6.1, C7.1, C8.1, D23.4 (VDD), D24.4 (VDD), D25.4 (VDD), D26.4 (VDD), D27.4 (VDD), D28.4 (VDD), D29.4 (VDD), D30.4 (VDD), D31.4 (VDD), D32.4 (VDD), D33.4 (VDD), D34.4 (VDD), D35.4 (VDD), D36.4 (VDD), D37.4 (VDD), D38.4 (VDD), D39.4 (VDD), D40.4 (VDD), D41.4 (VDD), D42.4 (VDD), D43.4 (VDD), D44.4 (VDD), D45.4 (VDD), D46.4 (VDD)
- net GND: now also C1.2, C2.2, C3.2, C4.2, C5.2, C6.2, C7.2, C8.2, D23.2 (VSS), D24.2 (VSS), D25.2 (VSS), D26.2 (VSS), D27.2 (VSS), D28.2 (VSS), D29.2 (VSS), D30.2 (VSS), D31.2 (VSS), D32.2 (VSS), D33.2 (VSS), D34.2 (VSS), D35.2 (VSS), D36.2 (VSS), D37.2 (VSS), D38.2 (VSS), D39.2 (VSS), D40.2 (VSS), D41.2 (VSS), D42.2 (VSS), D43.2 (VSS), D44.2 (VSS), D45.2 (VSS), D46.2 (VSS)
- new net: D23.1 (DOUT), D24.3 (DIN)
- new net: D25.1 (DOUT), D26.3 (DIN)
- new net: D24.1 (DOUT), D25.3 (DIN)
- new net: D27.1 (DOUT), D28.3 (DIN)
- new net: D26.1 (DOUT), D27.3 (DIN)
- new net: D34.1 (DOUT), D35.3 (DIN)
- new net: D33.1 (DOUT), D34.3 (DIN)
- new net: D30.1 (DOUT), D31.3 (DIN)
- new net: D29.1 (DOUT), D30.3 (DIN)
- new net: D45.1 (DOUT), D46.3 (DIN)
- new net: D44.1 (DOUT), D45.3 (DIN)
- new net: D37.1 (DOUT), D38.3 (DIN)
- new net: D36.1 (DOUT), D37.3 (DIN)
- new net: D39.1 (DOUT), D40.3 (DIN)
- new net: D38.1 (DOUT), D39.3 (DIN)
- new net: D28.1 (DOUT), D29.3 (DIN)
- new net: D32.1 (DOUT), D33.3 (DIN)
- new net: D31.1 (DOUT), D32.3 (DIN)
- new net: D35.1 (DOUT), D36.3 (DIN)
- new net: D43.1 (DOUT), D44.3 (DIN)
- new net: D42.1 (DOUT), D43.3 (DIN)
- new net: D40.1 (DOUT), D41.3 (DIN)
- new net: D41.1 (DOUT), D42.3 (DIN)
Other:
- moved on the sheet: D1, D10, D11, D12, D13, D14, D15, D16, D17, D18, D19, D2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

Commit message: pcb lights
Parts:
- removed D45, D46: SK6812MINI, LED_SMD:LED_SK6812MINI_PLCC4_3.5x3.5mm_P1.75mm, symbol LED:SK6812MINI
- C1, C2, C3, C4, C5, C6, C7, C8: footprint (none) -> Capacitor_SMD:C_1206_3216Metric
- D23, D24, D25, D26, D27, D28, D29, D30, D31, D32, D33, D34, D35, D36, D37, D38, D39, D40, D41, D42, D43, D44: footprint LED_SMD:LED_SK6812MINI_PLCC4_3.5x3.5mm_P1.75mm -> Keyboard:SK6812-MINI-E
Connections:
- net +5V: no longer J1.1
- net GND: no longer J1.2
- new net LED: J1.2
- no-connect marks 9 -> 11

Commit message: more traces
Connections:
- net LED: now also D23.3 (DIN); no longer J1.2
- new net LED_TXRX: J1.2
Changed lines of the file:
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@@
 	(wire
 		(pts
-			(xy 68.58 43.18) (xy 68.58 39.37)
+			(xy 73.66 43.18) (xy 73.66 39.37)
 		)
 		(stroke
@@
 	(wire
 		(pts
-			(xy 68.58 45.72) (xy 68.58 58.42)
+			(xy 73.66 45.72) (xy 73.66 58.42)
 		)
 		(stroke
@@
 	(wire
 		(pts
-			(xy 62.23 43.18) (xy 68.58 43.18)
+			(xy 62.23 43.18) (xy 73.66 43.18)
 		)
 		(stroke
@@
 	(wire
 		(pts
-			(xy 62.23 45.72) (xy 68.58 45.72)
+			(xy 62.23 45.72) (xy 73.66 45.72)
 		)
 		(stroke
@@
 		)
 	)
+	(label "LED"
+		(at 16.51 129.54 180)
+		(effects
+			(font
+				(size 1.27 1.27)
+			)
+			(justify right bottom)
+		)
+	)
 	(label "TX"
 		(at 63.5 50.8 0)
@@
 		)
 	)
-	(label "LED"
+	(label "LED_TXRX"
 		(at 63.5 53.34 0)
 		(effects
@@
 	(symbol
 		(lib_id "power:+5V")
-		(at 68.58 39.37 0)
+		(at 73.66 39.37 0)
 		(unit 1)
 		(exclude_from_sim no)
@@
 		(fields_autoplaced yes)
 		(property "Reference" "#PWR02"
-			(at 68.58 43.18 0)
+			(at 73.66 43.18 0)
 			(effects
 				(font
@@
 		)
 		(property "Value" "+5V"
-			(at 68.58 34.29 0)
+			(at 73.66 34.29 0)
 			(effects
 				(font
@@
 		)
 		(property "Footprint" ""
-			(at 68.58 39.37 0)
+			(at 73.66 39.37 0)
 			(effects
 				(font
@@
 		)
 		(property "Datasheet" ""
-			(at 68.58 39.37 0)
+			(at 73.66 39.37 0)
 			(effects
 				(font
@@
 		)
 		(property "Description" "Power symbol creates a global label with name \"+5V\""
-			(at 68.58 39.37 0)
+			(at 73.66 39.37 0)
 			(effects
 				(font
@@
 	(symbol
 		(lib_id "power:GND")
-		(at 68.58 58.42 0)
+		(at 73.66 58.42 0)
 		(unit 1)
 		(exclude_from_sim no)
@@
 		(fields_autoplaced yes)
 		(property "Reference" "#PWR01"
-			(at 68.58 64.77 0)
+			(at 73.66 64.77 0)
 			(effects
 				(font
@@
 		)
 		(property "Value" "GND"
-			(at 68.58 63.5 0)
+			(at 73.66 63.5 0)
 			(effects
 				(font
@@
 		)
 		(property "Footprint" ""
-			(at 68.58 58.42 0)
+			(at 73.66 58.42 0)
 			(effects
 				(font
@@
 		)
 		(property "Datasheet" ""
-			(at 68.58 58.42 0)
+			(at 73.66 58.42 0)
 			(effects
 				(font
@@
 		)
 		(property "Description" "Power symbol creates a global label with name \"GND\" , ground"
-			(at 68.58 58.42 0)
+			(at 73.66 58.42 0)
 			(effects
 				(font

Commit message: revisions
Parts:
- D1, D10, D11, D12, D13, D14, D15, D16, D17, D18, D19, D2, D20, D21, D22, D3, D4, D5, D6, D7, D8, D9: footprint Diode_SMD:D_SOD-123 -> Keyboard:D_SOD-128-Reversible
- SW1, SW10, SW11, SW12, SW13, SW14, SW15, SW16, SW17, SW18, SW19, SW2, SW20, SW21, SW22, SW3, SW4, SW5, SW6, SW7, SW8, SW9: footprint PCM_Switch_Keyboard_Hotswap_Kailh:SW_Hotswap_Kailh_Choc_V1V2_1.00u -> Keyboard:SW_Hotswap_Kailh_Choc_V1_1.00u
Changed lines of the file:
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@@
 			)
 		)
-		(property "Footprint" "Diode_SMD:D_SOD-123"
+		(property "Footprint" "Keyboard:D_SOD-128-Reversible"
 			(at 212.725 113.03 0)
 			(effects
@@
 			)
 		)
-		(property "Footprint" "Diode_SMD:D_SOD-123"
+		(property "Footprint" "Keyboard:D_SOD-128-Reversible"
 			(at 196.215 43.18 0)
 			(effects
@@
 			)
 		)
-		(property "Footprint" "PCM_Switch_Keyboard_Hotswap_Kailh:SW_Hotswap_Kailh_Choc_V1V2_1.00u"
+		(property "Footprint" "Keyboard:SW_Hotswap_Kailh_Choc_V1_1.00u"
 			(at 189.23 57.15 0)
 			(effects
@@
 			)
 		)
-		(property "Footprint" "Diode_SMD:D_SOD-123"
+		(property "Footprint" "Keyboard:D_SOD-128-Reversible"
 			(at 229.235 43.18 0)
 			(effects
@@
 			)
 		)
-		(property "Footprint" "PCM_Switch_Keyboard_Hotswap_Kailh:SW_Hotswap_Kailh_Choc_V1V2_1.00u"
+		(property "Footprint" "Keyboard:SW_Hotswap_Kailh_Choc_V1_1.00u"
 			(at 205.74 35.56 0)
 			(effects
@@
 			)
 		)
-		(property "Footprint" "PCM_Switch_Keyboard_Hotswap_Kailh:SW_Hotswap_Kailh_Choc_V1V2_1.00u"
+		(property "Footprint" "Keyboard:SW_Hotswap_Kailh_Choc_V1_1.00u"
 			(at 238.76 57.15 0)
 			(effects
@@
 			)
 		)
-		(property "Footprint" "Diode_SMD:D_SOD-123"
+		(property "Footprint" "Keyboard:D_SOD-128-Reversible"
 			(at 245.745 43.18 0)
 			(effects
@@
 			)
 		)
-		(property "Footprint" "Diode_SMD:D_SOD-123"
+		(property "Footprint" "Keyboard:D_SOD-128-Reversible"
 			(at 179.705 43.18 0)
 			(effects
@@
 			)
 		)
-		(property "Footprint" "Diode_SMD:D_SOD-123"
+		(property "Footprint" "Keyboard:D_SOD-128-Reversible"
 			(at 262.255 64.77 0)
 			(effects
@@
 			)
 		)
-		(property "Footprint" "Diode_SMD:D_SOD-123"
+		(property "Footprint" "Keyboard:D_SOD-128-Reversible"
 			(at 262.255 43.18 0)
 			(effects
@@
 			)
 		)
-		(property "Footprint" "Diode_SMD:D_SOD-123"
+		(property "Footprint" "Keyboard:D_SOD-128-Reversible"
 			(at 212.725 86.36 0)
 			(effects
@@
 			)
 		)
-		(property "Footprint" "PCM_Switch_Keyboard_Hotswap_Kailh:SW_Hotswap_Kailh_Choc_V1V2_1.00u"
+		(property "Footprint" "Keyboard:SW_Hotswap_Kailh_Choc_V1_1.00u"
 			(at 222.25 105.41 0)
 			(effects
@@
 			)
 		)
-		(property "Footprint" "Diode_SMD:D_SOD-123"
+		(property "Footprint" "Keyboard:D_SOD-128-Reversible"
 			(at 196.215 113.03 0)
 			(effects
@@
 			)
 		)
-		(property "Footprint" "Diode_SMD:D_SOD-123"
+		(property "Footprint" "Keyboard:D_SOD-128-Reversible"
 			(at 245.745 86.36 0)
 			(effects
@@
 			)
 		)
-		(property "Footprint" "Diode_SMD:D_SOD-123"
+		(property "Footprint" "Keyboard:D_SOD-128-Reversible"
 			(at 245.745 64.77 0)
 			(effects
@@
 			)
 		)
-		(property "Footprint" "PCM_Switch_Keyboard_Hotswap_Kailh:SW_Hotswap_Kailh_Choc_V1V2_1.00u"
+		(property "Footprint" "Keyboard:SW_Hotswap_Kailh_Choc_V1_1.00u"
 			(at 172.72 105.41 0)
 			(effects
@@
 			)
 		)
-		(property "Footprint" "Diode_SMD:D_SOD-123"
+		(property "Footprint" "Keyboard:D_SOD-128-Reversible"
 			(at 179.705 113.03 0)
 			(effects
@@
 			)
 		)
-		(property "Footprint" "Diode_SMD:D_SOD-123"
+		(property "Footprint" "Keyboard:D_SOD-128-Reversible"
 			(at 229.235 86.36 0)
 			(effects
@@
 			)
 		)
-		(property "Footprint" "PCM_Switch_Keyboard_Hotswap_Kailh:SW_Hotswap_Kailh_Choc_V1V2_1.00u"
+		(property "Footprint" "Keyboard:SW_Hotswap_Kailh_Choc_V1_1.00u"
 			(at 255.27 35.56 0)
 			(effects
@@
 			)
 		)
-		(property "Footprint" "Diode_SMD:D_SOD-123"
+		(property "Footprint" "Keyboard:D_SOD-128-Reversible"
 			(at 179.705 64.77 0)
 			(effects
@@
 			)
 		)
-		(property "Footprint" "Diode_SMD:D_SOD-123"
+		(property "Footprint" "Keyboard:D_SOD-128-Reversible"
 			(at 179.705 86.36 0)
 			(effects
@@
 			)
 		)
-		(property "Footprint" "PCM_Switch_Keyboard_Hotswap_Kailh:SW_Hotswap_Kailh_Choc_V1V2_1.00u"
+		(property "Footprint" "Keyboard:SW_Hotswap_Kailh_Choc_V1_1.00u"
 			(at 189.23 35.56 0)
 			(effects
@@
 			)
 		)
-		(property "Footprint" "PCM_Switch_Keyboard_Hotswap_Kailh:SW_Hotswap_Kailh_Choc_V1V2_1.00u"
+		(property "Footprint" "Keyboard:SW_Hotswap_Kailh_Choc_V1_1.00u"
 			(at 222.25 35.56 0)
 			(effects
@@
 			)
 		)
-		(property "Footprint" "PCM_Switch_Keyboard_Hotswap_Kailh:SW_Hotswap_Kailh_Choc_V1V2_1.00u"
+		(property "Footprint" "Keyboard:SW_Hotswap_Kailh_Choc_V1_1.00u"
 			(at 255.27 57.15 0)
 			(effects
@@
 			)
 		)
-		(property "Footprint" "Diode_SMD:D_SOD-123"
+		(property "Footprint" "Keyboard:D_SOD-128-Reversible"
 			(at 262.255 86.36 0)
 			(effects
@@
 			)
 		)
-		(property "Footprint" "PCM_Switch_Keyboard_Hotswap_Kailh:SW_Hotswap_Kailh_Choc_V1V2_1.00u"
+		(property "Footprint" "Keyboard:SW_Hotswap_Kailh_Choc_V1_1.00u"
 			(at 172.72 35.56 0)
 			(effects
@@
 			)
 		)
-		(property "Footprint" "PCM_Switch_Keyboard_Hotswap_Kailh:SW_Hotswap_Kailh_Choc_V1V2_1.00u"
+		(property "Footprint" "Keyboard:SW_Hotswap_Kailh_Choc_V1_1.00u"
 			(at 189.23 78.74 0)
 			(effects
@@
 			)
 		)
-		(property "Footprint" "Diode_SMD:D_SOD-123"
+		(property "Footprint" "Keyboard:D_SOD-128-Reversible"
 			(at 212.725 64.77 0)
 			(effects
@@
 			)
 		)
-		(property "Footprint" "PCM_Switch_Keyboard_Hotswap_Kailh:SW_Hotswap_Kailh_Choc_V1V2_1.00u"
+		(property "Footprint" "Keyboard:SW_Hotswap_Kailh_Choc_V1_1.00u"
 			(at 205.74 105.41 0)
 			(effects
@@
 			)
 		)
-		(property "Footprint" "PCM_Switch_Keyboard_Hotswap_Kailh:SW_Hotswap_Kailh_Choc_V1V2_1.00u"
+		(property "Footprint" "Keyboard:SW_Hotswap_Kailh_Choc_V1_1.00u"
 			(at 222.25 57.15 0)
 			(effects
@@
 			)
 		)
-		(property "Footprint" "PCM_Switch_Keyboard_Hotswap_Kailh:SW_Hotswap_Kailh_Choc_V1V2_1.00u"
+		(property "Footprint" "Keyboard:SW_Hotswap_Kailh_Choc_V1_1.00u"
 			(at 238.76 35.56 0)
 			(effects
@@
 			)
 		)
-		(property "Footprint" "Diode_SMD:D_SOD-123"
+		(property "Footprint" "Keyboard:D_SOD-128-Reversible"
 			(at 229.235 113.03 0)
 			(effects
@@
 			)
 		)
-		(property "Footprint" "PCM_Switch_Keyboard_Hotswap_Kailh:SW_Hotswap_Kailh_Choc_V1V2_1.00u"
+		(property "Footprint" "Keyboard:SW_Hotswap_Kailh_Choc_V1_1.00u"
 			(at 238.76 78.74 0)
 			(effects
@@
 			)
 		)
-		(property "Footprint" "PCM_Switch_Keyboard_Hotswap_Kailh:SW_Hotswap_Kailh_Choc_V1V2_1.00u"
+		(property "Footprint" "Keyboard:SW_Hotswap_Kailh_Choc_V1_1.00u"
 			(at 189.23 105.41 0)
 			(effects
@@
 			)
 		)
-		(property "Footprint" "Diode_SMD:D_SOD-123"
+		(property "Footprint" "Keyboard:D_SOD-128-Reversible"
 			(at 212.725 43.18 0)
 			(effects
@@
 			)
 		)
-		(property "Footprint" "Diode_SMD:D_SOD-123"
+		(property "Footprint" "Keyboard:D_SOD-128-Reversible"
 			(at 196.215 86.36 0)
 			(effects
@@
 			)
 		)
-		(property "Footprint" "PCM_Switch_Keyboard_Hotswap_Kailh:SW_Hotswap_Kailh_Choc_V1V2_1.00u"
+		(property "Footprint" "Keyboard:SW_Hotswap_Kailh_Choc_V1_1.00u"
 			(at 222.25 78.74 0)
 			(effects
@@
 			)
 		)
-		(property "Footprint" "PCM_Switch_Keyboard_Hotswap_Kailh:SW_Hotswap_Kailh_Choc_V1V2_1.00u"
+		(property "Footprint" "Keyboard:SW_Hotswap_Kailh_Choc_V1_1.00u"
 			(at 172.72 78.74 0)
 			(effects
@@
 			)
 		)
-		(property "Footprint" "PCM_Switch_Keyboard_Hotswap_Kailh:SW_Hotswap_Kailh_Choc_V1V2_1.00u"
+		(property "Footprint" "Keyboard:SW_Hotswap_Kailh_Choc_V1_1.00u"
 			(at 205.74 78.74 0)
 			(effects
@@
 			)
 		)
-		(property "Footprint" "Diode_SMD:D_SOD-123"
+		(property "Footprint" "Keyboard:D_SOD-128-Reversible"
 			(at 196.215 64.77 0)
 			(effects
@@
 			)
 		)
-		(property "Footprint" "PCM_Switch_Keyboard_Hotswap_Kailh:SW_Hotswap_Kailh_Choc_V1V2_1.00u"
+		(property "Footprint" "Keyboard:SW_Hotswap_Kailh_Choc_V1_1.00u"
 			(at 255.27 78.74 0)
 			(effects
@@
 			)
 		)
-		(property "Footprint" "PCM_Switch_Keyboard_Hotswap_Kailh:SW_Hotswap_Kailh_Choc_V1V2_1.00u"
+		(property "Footprint" "Keyboard:SW_Hotswap_Kailh_Choc_V1_1.00u"
 			(at 172.72 57.15 0)
 			(effects
@@
 			)
 		)
-		(property "Footprint" "PCM_Switch_Keyboard_Hotswap_Kailh:SW_Hotswap_Kailh_Choc_V1V2_1.00u"
+		(property "Footprint" "Keyboard:SW_Hotswap_Kailh_Choc_V1_1.00u"
 			(at 205.74 57.15 0)
 			(effects
@@
 			)
 		)
-		(property "Footprint" "Diode_SMD:D_SOD-123"
+		(property "Footprint" "Keyboard:D_SOD-128-Reversible"
 			(at 229.235 64.77 0)
 			(effects

Commit message: revisions
Connections:
- net LED_TXRX: now also U1.9 (GP9)
- no-connect marks 11 -> 10
Changed lines of the file:
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@@
-	)
-	(no_connect
-		(at 104.14 68.58)
 	)
 	(no_connect
@@
 		(pts
 			(xy 186.69 33.02) (xy 186.69 54.61)
+		)
+		(stroke
+			(width 0)
+			(type default)
+		)
+	)
+	(wire
+		(pts
+			(xy 102.87 68.58) (xy 104.14 68.58)
 		)
 		(stroke
@@
 		)
 	)
+	(label "LED_TXRX"
+		(at 102.87 68.58 180)
+		(effects
+			(font
+				(size 1.27 1.27)
+			)
+			(justify right bottom)
+		)
+	)

Commit message: revisions
Parts:
- C1, C2, C3, C4, C5, C6, C7, C8: footprint Capacitor_SMD:C_1206_3216Metric -> Keyboard:C_1206_3216Metric
Changed lines of the file:
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@@
 			)
 		)
-		(property "Footprint" "Capacitor_SMD:C_1206_3216Metric"
+		(property "Footprint" "Keyboard:C_1206_3216Metric"
 			(at 173.99 120.65 0)
 			(effects
@@
 			)
 		)
-		(property "Footprint" "Capacitor_SMD:C_1206_3216Metric"
+		(property "Footprint" "Keyboard:C_1206_3216Metric"
 			(at 193.04 148.59 0)
 			(effects
@@
 			)
 		)
-		(property "Footprint" "Capacitor_SMD:C_1206_3216Metric"
+		(property "Footprint" "Keyboard:C_1206_3216Metric"
 			(at 86.36 148.59 0)
 			(effects
@@
 			)
 		)
-		(property "Footprint" "Capacitor_SMD:C_1206_3216Metric"
+		(property "Footprint" "Keyboard:C_1206_3216Metric"
 			(at 13.97 121.92 0)
 			(effects
@@
 			)
 		)
-		(property "Footprint" "Capacitor_SMD:C_1206_3216Metric"
+		(property "Footprint" "Keyboard:C_1206_3216Metric"
 			(at 139.7 148.59 0)
 			(effects
@@
 			)
 		)
-		(property "Footprint" "Capacitor_SMD:C_1206_3216Metric"
+		(property "Footprint" "Keyboard:C_1206_3216Metric"
 			(at 67.31 120.65 0)
 			(effects
@@
 			)
 		)
-		(property "Footprint" "Capacitor_SMD:C_1206_3216Metric"
+		(property "Footprint" "Keyboard:C_1206_3216Metric"
 			(at 27.94 148.59 0)
 			(effects
@@
 			)
 		)
-		(property "Footprint" "Capacitor_SMD:C_1206_3216Metric"
+		(property "Footprint" "Keyboard:C_1206_3216Metric"
 			(at 120.65 120.65 0)
 			(effects

Commit message: level shifter
Parts:
- added R1: 500, Keyboard:R_Axial_DIN0207_L6.3mm_D2.5mm_P7.62mm_Horizontal, symbol Device:R
- added U2: SN74LV1T34DBV, Keyboard:SOT-23-5, symbol Logic_LevelTranslator:SN74LV1T34DBV
Connections:
- net +5V: now also U2.5 (VCC)
- net GND: now also J1.1, U2.3 (GND)
- net LED: now also U1.21 (GP21), R1.2; no longer D23.3 (DIN)
- net LED_TX: now reaches D44.1 (DOUT)
- net LED_TX: now also J1.2
- net LED_TXRX: no longer names the net of U1.9 (GP9)
- net LED_TXRX: no longer J1.2
- new net: D23.3 (DIN), U2.4 (Y)
- new net: R1.1, U2.2 (A)
- no-connect marks 10 -> 8
Other:
- note added: "Note: This schematic is for the master half (left side). For the slave half, the GP21 pin is unconnected, and pin 2 of J1 is connected to LED. Lastly, pin 1 of D44 is disconnected."

Commit message: maybe functional
Parts:
- U2: footprint Keyboard:SOT-23-5 -> Package_TO_SOT_SMD:SOT-23-5
Other:
- note added: "Note: This schematic is for the master half (left side). For the slave half, the GP21 pin is unconnected, and pin 2 of J1 is connected to pin 3 of D23 (bypassing the resistor and level shifter). Lastly, pin 1 of D44 is disconnected."
- note removed: "Note: This schematic is for the master half (left side). For the slave half, the GP21 pin is unconnected, and pin 2 of J1 is connected to LED. Lastly, pin 1 of D44 is disconnected."
Changed lines of the file:
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@@
 	(generator_version "9.0")
 	(paper "A4")
-	(text "Note: This schematic is for the master half (left side).\nFor the slave half, the GP21 pin is unconnected,\nand pin 2 of J1 is connected to LED.\nLastly, pin 1 of D44 is disconnected."
+	(text "Note: This schematic is for the master half (left side).\nFor the slave half, the GP21 pin is unconnected,\nand pin 2 of J1 is connected to pin 3 of D23\n(bypassing the resistor and level shifter).\nLastly, pin 1 of D44 is disconnected."
 		(exclude_from_sim no)
-		(at 112.776 93.726 0)
+		(at 76.454 90.678 0)
 		(effects
 			(font
 				(size 1.27 1.27)
 			)
+			(justify left)
 		)
 	)
@@
 			)
 		)
-		(property "Footprint" "Keyboard:SOT-23-5"
+		(property "Footprint" "Package_TO_SOT_SMD:SOT-23-5"
 			(at 20.32 87.63 0)
 			(effects
