File: astronomer.kicad_sch (KiCad schematic)
At the start: 78 parts, among them J1 6P6C, SW1 SW_Push_45deg, SW10 SW_Push_45deg, SW11 SW_Push_45deg, SW12 SW_Push_45deg, SW13 SW_Push_45deg, SW14 SW_Push_45deg, SW15 SW_Push_45deg, SW16 SW_Push_45deg, SW17 SW_Push_45deg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

Commit message: added the footprints + symbols
Parts:
- C1, C2, C3, C4, C5, C6, C7, C8: symbol Device:C_Small -> library:C_Small
- D1, D10, D11, D12, D13, D14, D15, D16, D17, D18, D19, D2, D20, D21, D22, D3, D4, D5, D6, D7, D8, D9: symbol Diode:1N4148W -> library:1N4148W
- D23, D24, D25, D26, D27, D28, D29, D30, D31, D32, D33, D34, D35, D36, D37, D38, D39, D40, D41, D42, D43, D44: symbol LED:SK6812MINI -> library:SK6812MINI
- J1: symbol Connector:6P6C -> library:6P6C
- R1: symbol Device:R -> library:R
- SW1, SW10, SW11, SW12, SW13, SW14, SW15, SW16, SW17, SW18, SW19, SW2, SW20, SW21, SW22, SW3, SW4, SW5, SW6, SW7, SW8, SW9: symbol Switch:SW_Push_45deg -> library:SW_Push_45deg
- U1: symbol Keyboard:RP2040_ProMicro -> library:RP2040_ProMicro
- U2: symbol Logic_LevelTranslator:SN74LV1T34DBV -> library:SN74LV1T34DBV

Commit message: Probably works
Parts:
- D1, D10, D11, D12, D13, D14, D15, D16, D17, D18, D19, D2, D20, D21, D22, D3, D4, D5, D6, D7, D8, D9: footprint Keyboard:D_SOD-128-Reversible -> Library:D_SOD-123 Reversible
Changed lines of the file:
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@@
 			)
 		)
-		(property "Footprint" "Keyboard:D_SOD-128-Reversible"
+		(property "Footprint" "Library:D_SOD-123 Reversible"
 			(at 212.725 113.03 0)
 			(effects
@@
 			)
 		)
-		(property "Footprint" "Keyboard:D_SOD-128-Reversible"
+		(property "Footprint" "Library:D_SOD-123 Reversible"
 			(at 196.215 43.18 0)
 			(effects
@@
 			)
 		)
-		(property "Footprint" "Keyboard:D_SOD-128-Reversible"
+		(property "Footprint" "Library:D_SOD-123 Reversible"
 			(at 229.235 43.18 0)
 			(effects
@@
 			)
 		)
-		(property "Footprint" "Keyboard:D_SOD-128-Reversible"
+		(property "Footprint" "Library:D_SOD-123 Reversible"
 			(at 245.745 43.18 0)
 			(effects
@@
 			)
 		)
-		(property "Footprint" "Keyboard:D_SOD-128-Reversible"
+		(property "Footprint" "Library:D_SOD-123 Reversible"
 			(at 179.705 43.18 0)
 			(effects
@@
 			)
 		)
-		(property "Footprint" "Keyboard:D_SOD-128-Reversible"
+		(property "Footprint" "Library:D_SOD-123 Reversible"
 			(at 262.255 64.77 0)
 			(effects
@@
 			)
 		)
-		(property "Footprint" "Keyboard:D_SOD-128-Reversible"
+		(property "Footprint" "Library:D_SOD-123 Reversible"
 			(at 262.255 43.18 0)
 			(effects
@@
 			)
 		)
-		(property "Footprint" "Keyboard:D_SOD-128-Reversible"
+		(property "Footprint" "Library:D_SOD-123 Reversible"
 			(at 212.725 86.36 0)
 			(effects
@@
 			)
 		)
-		(property "Footprint" "Keyboard:D_SOD-128-Reversible"
+		(property "Footprint" "Library:D_SOD-123 Reversible"
 			(at 196.215 113.03 0)
 			(effects
@@
 			)
 		)
-		(property "Footprint" "Keyboard:D_SOD-128-Reversible"
+		(property "Footprint" "Library:D_SOD-123 Reversible"
 			(at 245.745 86.36 0)
 			(effects
@@
 			)
 		)
-		(property "Footprint" "Keyboard:D_SOD-128-Reversible"
+		(property "Footprint" "Library:D_SOD-123 Reversible"
 			(at 245.745 64.77 0)
 			(effects
@@
 			)
 		)
-		(property "Footprint" "Keyboard:D_SOD-128-Reversible"
+		(property "Footprint" "Library:D_SOD-123 Reversible"
 			(at 179.705 113.03 0)
 			(effects
@@
 			)
 		)
-		(property "Footprint" "Keyboard:D_SOD-128-Reversible"
+		(property "Footprint" "Library:D_SOD-123 Reversible"
 			(at 229.235 86.36 0)
 			(effects
@@
 			)
 		)
-		(property "Footprint" "Keyboard:D_SOD-128-Reversible"
+		(property "Footprint" "Library:D_SOD-123 Reversible"
 			(at 179.705 64.77 0)
 			(effects
@@
 			)
 		)
-		(property "Footprint" "Keyboard:D_SOD-128-Reversible"
+		(property "Footprint" "Library:D_SOD-123 Reversible"
 			(at 179.705 86.36 0)
 			(effects
@@
 			)
 		)
-		(property "Footprint" "Keyboard:D_SOD-128-Reversible"
+		(property "Footprint" "Library:D_SOD-123 Reversible"
 			(at 262.255 86.36 0)
 			(effects
@@
 			)
 		)
-		(property "Footprint" "Keyboard:D_SOD-128-Reversible"
+		(property "Footprint" "Library:D_SOD-123 Reversible"
 			(at 212.725 64.77 0)
 			(effects
@@
 			)
 		)
-		(property "Footprint" "Keyboard:D_SOD-128-Reversible"
+		(property "Footprint" "Library:D_SOD-123 Reversible"
 			(at 229.235 113.03 0)
 			(effects
@@
 			)
 		)
-		(property "Footprint" "Keyboard:D_SOD-128-Reversible"
+		(property "Footprint" "Library:D_SOD-123 Reversible"
 			(at 212.725 43.18 0)
 			(effects
@@
 			)
 		)
-		(property "Footprint" "Keyboard:D_SOD-128-Reversible"
+		(property "Footprint" "Library:D_SOD-123 Reversible"
 			(at 196.215 86.36 0)
 			(effects
@@
 			)
 		)
-		(property "Footprint" "Keyboard:D_SOD-128-Reversible"
+		(property "Footprint" "Library:D_SOD-123 Reversible"
 			(at 196.215 64.77 0)
 			(effects
@@
 			)
 		)
-		(property "Footprint" "Keyboard:D_SOD-128-Reversible"
+		(property "Footprint" "Library:D_SOD-123 Reversible"
 			(at 229.235 64.77 0)
 			(effects
