File: astronomer.kicad_pcb (KiCad board)
At the start: 2 copper layers, 160.9 x 114.4 mm, 76 parts, among them J1 6P6C, SW1 SW_Push_45deg, SW10 SW_Push_45deg, SW11 SW_Push_45deg, SW12 SW_Push_45deg, SW13 SW_Push_45deg, SW14 SW_Push_45deg, SW15 SW_Push_45deg, SW16 SW_Push_45deg, SW17 SW_Push_45deg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

Commit message: revisions
Parts:
- added REF**: MountingHole_2.2mm_M2, MountingHole:MountingHole_2.2mm_M2, F.Cu at (143.8, 51.7)
- added REF**: MountingHole_2.2mm_M2, MountingHole:MountingHole_2.2mm_M2, F.Cu at (151.1, 83.2)
- added REF**: MountingHole_2.2mm_M2, MountingHole:MountingHole_2.2mm_M2, F.Cu at (178.2, 100.5)
- added REF**: MountingHole_2.2mm_M2, MountingHole:MountingHole_2.2mm_M2, F.Cu at (248.1, 104.3)
- added REF**: MountingHole_2.2mm_M2, MountingHole:MountingHole_2.2mm_M2, F.Cu at (254.2, 48.6)
- moved D16 59.8 mm to (223.3, 97.8), turned to -90 degrees
- moved D9 59.8 mm to (200.5, 94.9), turned to 90 degrees
- moved D15 59.7 mm to (220.1, 97.8), turned to -90 degrees
- moved D10 59.7 mm to (203.8, 94.9), turned to 90 degrees
- moved D14 59.7 mm to (216.8, 97.8), turned to -90 degrees
- moved D11 59.7 mm to (207.0, 94.9), turned to 90 degrees
- moved D13 59.6 mm to (213.6, 97.8), turned to -90 degrees
- moved D12 59.6 mm to (210.3, 94.9)
- moved D7 56.6 mm to (194.0, 96.6)
- moved D8 54.8 mm to (197.2, 94.9), turned to 90 degrees
- moved D18 53.6 mm to (229.9, 97.8), turned to -90 degrees
- moved D17 53.4 mm to (226.6, 97.8), turned to -90 degrees
- moved C4 11.7 mm to (214.9, 62.5), turned to 180 degrees
- moved D6 8.58 mm to (174.7, 45.7)
- moved D5 7.78 mm to (171.2, 45.7)
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
Commit message: revisions
Parts:
- C1, C2, C3, C4, C5, C6, C7, C8: footprint Capacitor_SMD:C_1206_3216Metric -> Keyboard:C_1206_3216Metric
- moved D6 71.6 mm to (246.2, 46.1), turned to -30 degrees
- moved D5 68.7 mm to (240.0, 46.1), turned to -30 degrees
- moved D4 65.9 mm to (233.7, 46.1), turned to -30 degrees
- moved D3 7.88 mm to (172.3, 46.1), turned to -150 degrees
- moved D2 5.06 mm to (166.0, 46.1), turned to -150 degrees
- moved D1 2.41 mm to (160.0, 46.1), turned to -150 degrees
- moved C7 1.26 mm to (188.2, 102.2)
- moved REF** 1.12 mm to (143.8, 52.8)
- moved D44 1.08 mm to (142.0, 96.3)
- moved D43 0.92 mm to (144.1, 116.3)
- moved D42 0.89 mm to (165.9, 107.8)
- moved D41 0.86 mm to (189.9, 106.3)
- moved D30 0.84 mm to (241.6, 69.2)
- moved D33 0.84 mm to (184.5, 64.7)
- moved D34 0.84 mm to (165.6, 69.2)
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Connections:
- U1 pad 9: unconnected-(U1-GP9-Pad9)_1 -> /LED_TXRX
Routing:
- net +5V: track 0.00 -> 872.1 mm, vias 0 -> 49
- net /Col 6: track 0.00 -> 254.2 mm, vias 0 -> 8
- net /Col 5: track 0.00 -> 226.6 mm, vias 0 -> 7
- net /Col 3: track 0.00 -> 202.8 mm, vias 0 -> 6
- net /Col 4: track 0.00 -> 199.8 mm, vias 0 -> 8
- net /Col 2: track 0.00 -> 155.5 mm, vias 0 -> 9
- net /Col 1: track 0.00 -> 134.1 mm, vias 0 -> 8
- net /Row 1: track 0.00 -> 131.0 mm, vias 0 -> 8
- net /Row 3: track 0.00 -> 112.1 mm, vias 0 -> 7
- net /Row 2: track 0.00 -> 101.0 mm, vias 0 -> 7
- net GND: track 0.00 -> 88.7 mm, vias 0 -> 33
- net Net-(D40-DOUT): track 0.00 -> 88.1 mm, vias 0 -> 5
- net Net-(D13-A): track 0.00 -> 81.1 mm, vias 0 -> 2
- net Net-(D22-A): track 0.00 -> 73.3 mm, vias 0 -> 2
- net /Row 4: track 0.00 -> 72.0 mm, vias 0 -> 7
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- added copper zone on F.Cu, net GND
Other:
- board text added: "M"
- board text added: "S"

Commit message: routes done?
Routing:
- net /LED: track 8.08 -> 72.9 mm, vias 1 -> 3
- net /Col 2: track 155.5 -> 204.4 mm, vias 9 -> 16
- net +5V: track 872.1 -> 893.5 mm, vias 49 -> 51
- net Net-(D8-A): track 31.8 -> 50.8 mm, vias 1 -> 2
- net /LED_TXRX: track 25.7 -> 42.1 mm, vias 0 -> 2
- net /Row 3: track 112.1 -> 124.8 mm, vias 7 -> 15
- net Net-(D25-DOUT): track 21.0 -> 29.1 mm, vias 3 -> 4
- net /Col 4: track 199.8 -> 207.8 mm, vias 8 -> 9
- net Net-(D24-DOUT): track 38.9 -> 32.0 mm, vias 3 -> 4
- net Net-(D34-DOUT): track 36.0 -> 39.9 mm, vias 5 -> 6
- net /Col 1: track 134.1 -> 137.4 mm
- net Net-(D33-DOUT): track 38.0 -> 36.2 mm
- net /Row 2: track 101.0 -> 102.4 mm, vias 7 -> 13
- net GND: track 88.7 -> 89.9 mm
- net Net-(D40-DOUT): track 88.1 -> 88.2 mm, vias 5 -> 7
Other:
- board size 160.9 x 114.4 mm -> 148 x 98.6 mm

Commit message: level shifter
Parts:
- removed the REF** at (143.8, 52.8)
- removed the REF** at (151.1, 83.2)
- removed the REF** at (178.2, 100.5)
- removed the REF** at (248.1, 104.3)
- removed the REF** at (254.2, 48.6)
- added R1: 500, Keyboard:R_Axial_DIN0207_L6.3mm_D2.5mm_P7.62mm_Horizontal, F.Cu at (144.1, 79.1)
- added REF**: MountingHole_2.2mm_M2, Keyboard:MountingHole_2.2mm_M2, F.Cu at (151.1, 83.2)
- added REF**: MountingHole_2.2mm_M2, Keyboard:MountingHole_2.2mm_M2, F.Cu at (248.1, 104.3)
- added REF**: MountingHole_2.2mm_M2, Keyboard:MountingHole_2.2mm_M2, F.Cu at (254.2, 48.6)
- added REF**: MountingHole_2.2mm_M2, Keyboard:MountingHole_2.2mm_M2, F.Cu at (143.8, 52.8)
- added REF**: MountingHole_2.2mm_M2, Keyboard:MountingHole_2.2mm_M2, F.Cu at (178.2, 100.5)
- added U2: SN74LV1T34DBV, Keyboard:SOT-23-5, F.Cu at (143.2, 44.0)
- moved C7 0.71 mm to (187.7, 101.6)
Connections:
- D23 pad 3: /LED -> Net-(D23-DIN)
- D44 pad 1: unconnected-(D44-DOUT-Pad1)_1 -> /LED_TX
- J1 pad 1: unconnected-(J1-Pad1) -> GND
- J1 pad 2: /LED_TXRX -> /LED_TX
- U1 pad 21: unconnected-(U1-GP21-Pad21) -> /LED
- U1 pad 9: /LED_TXRX -> unconnected-(U1-GP9-Pad9)
Routing:
- net /LED_TXRX: track 42.1 -> 0.00 mm, vias 2 -> 0
- net /LED: track 72.9 -> 33.1 mm, vias 3 -> 0
- net Net-(U2-A): track 0.00 -> 39.7 mm, vias 0 -> 2
- net Net-(D23-DIN): track 0.00 -> 33.5 mm, vias 0 -> 6
- net /LED_TX: track 0.00 -> 7.06 mm, vias 0 -> 1
- net +5V: track 893.5 -> 896.7 mm, vias 51 -> 52
- net /Col 3: track 202.8 -> 203.5 mm
- net Net-(D13-A): track 81.1 -> 81.7 mm
- net Net-(D20-A): track 46.7 -> 46.4 mm, vias 2 -> 4
- net GND: vias 33 -> 34
Other:
- board size 148 x 98.6 mm -> 148 x 98.4 mm

Commit message: maybe functional
Parts:
- U2: footprint Keyboard:SOT-23-5 -> Package_TO_SOT_SMD:SOT-23-5; moved to B.Cu
- moved R1 7.32 mm to (151.5, 79.1), turned to 180 degrees
- turned U2 to 0 degrees
Routing:
- net Net-(D23-DIN): track 33.5 -> 102.7 mm, vias 6 -> 7
- net /LED: track 33.1 -> 6.80 mm
- net +5V: track 896.7 -> 900.2 mm, vias 52 -> 51
- net /Col 4: track 207.8 -> 204.6 mm
- net GND: track 89.9 -> 91.4 mm
- net Net-(U2-A): track 39.7 -> 41.2 mm, vias 2 -> 4
Other:
- outline, holes or cut-outs redrawn

Commit message: minor fixes
Parts:
- moved J1 3.28 mm to (123.3, 79.3)
Routing:
- net GND: track 91.4 -> 44.9 mm, vias 34 -> 31
- net /Row 1: track 131.3 -> 141.3 mm, vias 8 -> 13
- net Net-(D43-DOUT): track 37.9 -> 32.5 mm, vias 4 -> 3
- net Net-(D23-DIN): track 102.7 -> 107.5 mm, vias 7 -> 11
- net /Row 4: track 72.0 -> 75.7 mm
- net +5V: track 900.2 -> 898.4 mm
- net /TX: track 68.4 -> 69.6 mm, vias 0 -> 1
- net /LED_TX: track 7.06 -> 6.31 mm, vias 1 -> 0
- net /RX: track 65.1 -> 64.7 mm, vias 1 -> 0
- added copper zone on B.Cu, net (none)
Other:
- board size 148 x 98.4 mm -> 150.7 x 99.3 mm
