File: astronomer.kicad_pcb (KiCad board)
At the start: 2 copper layers, 150.7 x 99.3 mm, 83 parts, among them J1 6P6C, SW1 SW_Push_45deg, SW10 SW_Push_45deg, SW11 SW_Push_45deg, SW12 SW_Push_45deg, SW13 SW_Push_45deg, SW14 SW_Push_45deg, SW15 SW_Push_45deg, SW16 SW_Push_45deg, SW17 SW_Push_45deg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

Commit message: added the footprints + symbols
Parts:
- C1, C2, C3, C4, C5, C6, C7, C8: footprint Keyboard:C_1206_3216Metric -> footprints:C_1206_3216Metric
- D1, D10, D11, D12, D13, D14, D15, D16, D17, D18, D19, D2, D20, D21, D22, D3, D4, D5, D6, D7, D8, D9: footprint Keyboard:D_SOD-128-Reversible -> footprints:D_SOD-128-Reversible
- D23, D24, D25, D26, D27, D28, D29, D30, D31, D32, D33, D34, D35, D36, D37, D38, D39, D40, D41, D42, D43, D44: footprint Keyboard:SK6812-MINI-E -> footprints:SK6812-MINI-E
- J1: footprint Keyboard:RJ12 6P6C -> footprints:RJ12 6P6C
- R1: footprint Keyboard:R_Axial_DIN0207_L6.3mm_D2.5mm_P7.62mm_Horizontal -> footprints:R_Axial_DIN0207_L6.3mm_D2.5mm_P7.62mm_Horizontal
- REF** (x5): footprint Keyboard:MountingHole_2.2mm_M2 -> footprints:MountingHole_2.2mm_M2
- SW1, SW10, SW11, SW12, SW13, SW14, SW15, SW16, SW17, SW18, SW19, SW2, SW20, SW21, SW22, SW3, SW4, SW5, SW6, SW7, SW8, SW9: footprint Keyboard:SW_Hotswap_Kailh_Choc_V1_1.00u -> footprints:SW_Hotswap_Kailh_Choc_V1_1.00u
- U1: footprint Keyboard:RP2040_ProMicro -> footprints:RP2040_ProMicro
- U2: footprint Package_TO_SOT_SMD:SOT-23-5 -> footprints:SOT-23-5

Commit message: Probably works
Parts:
- D1, D10, D12, D13, D14, D15, D16, D17, D18, D19, D2, D20, D21, D22, D3, D4, D5, D6, D7, D8, D9: footprint footprints:D_SOD-128-Reversible -> Library:D_SOD-123 Reversible; moved to F.Cu
- D11: footprint footprints:D_SOD-128-Reversible -> Library:D_SOD-123 Reversible
- U2: footprint footprints:SOT-23-5 -> Package_TO_SOT_SMD:SOT-23-5
- moved D22 5.65 mm to (136.9, 108.3)
- moved D21 3.23 mm to (134.6, 109.6)
- moved D20 2.09 mm to (131.1, 105.6)
- moved D19 1.75 mm to (133.4, 104.3)
- moved D12 0.85 mm to (209.8, 94.2)
- moved D14 0.84 mm to (216.2, 97.2)
- moved D15 0.81 mm to (219.6, 97.2)
- moved D13 0.79 mm to (213.1, 97.2)
- moved D16 0.79 mm to (222.8, 97.2)
- moved D9 0.78 mm to (199.9, 94.3)
- moved D18 0.78 mm to (229.3, 97.3)
- moved D11 0.77 mm to (207.6, 94.3)
- moved D4 0.76 mm to (233.4, 45.4)
- moved D2 0.76 mm to (166.8, 46.2)
- moved D10 0.75 mm to (203.2, 94.3)
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Routing:
- net Net-(D43-DOUT): track 32.5 -> 37.4 mm, vias 3 -> 4
- net Net-(D21-A): track 43.8 -> 48.0 mm, vias 2 -> 3
- net /Row 4: track 75.7 -> 71.7 mm, vias 7 -> 6
- net Net-(D6-A): track 38.3 -> 39.5 mm
- net Net-(D22-A): track 73.3 -> 72.4 mm, vias 2 -> 6
- net Net-(D4-A): track 34.1 -> 33.2 mm
- net Net-(D19-A): track 28.8 -> 29.6 mm, vias 2 -> 3
- net Net-(D5-A): track 37.2 -> 36.4 mm
- net /Row 3: track 124.8 -> 125.5 mm
- net Net-(D2-A): track 35.3 -> 34.6 mm
- net /Row 2: track 102.4 -> 103.0 mm
- net Net-(D7-A): track 50.4 -> 51.0 mm

Commit message: Initial routing
Parts:
- moved D6 7.88 mm to (238.2, 46.4), turned to -90 degrees
- moved D3 7.66 mm to (165.3, 46.4), turned to -90 degrees
- moved D5 4.52 mm to (235.3, 46.4), turned to -90 degrees
- moved D2 4.36 mm to (162.5, 46.4), turned to -90 degrees
- moved D7 3.59 mm to (195.9, 94.0)
- moved D20 3.47 mm to (131.2, 102.1)
- moved D21 3.47 mm to (134.7, 106.1)
- moved D19 3.47 mm to (133.5, 100.8)
- moved D22 3.47 mm to (137.0, 104.8)
- moved D8 2.02 mm to (198.7, 94.0)
- moved D13 1.91 mm to (214.9, 97.0)
- moved D14 1.59 mm to (217.8, 97.0)
- moved D9 1.52 mm to (201.4, 94.0)
- moved D4 1.44 mm to (232.4, 46.4), turned to -90 degrees
- moved D38 1.30 mm to (222.6, 81.7)
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Routing:
- net +5V: track 898.4 -> 0.00 mm, vias 51 -> 0
- net /Col 6: track 254.5 -> 38.8 mm, vias 8 -> 4
- net /Col 5: track 227.0 -> 38.6 mm, vias 7 -> 3
- net /Col 4: track 204.6 -> 46.7 mm, vias 9 -> 4
- net /Col 2: track 204.4 -> 46.5 mm, vias 16 -> 4
- net /Col 3: track 203.5 -> 46.1 mm, vias 6 -> 4
- net /Row 1: track 141.3 -> 29.1 mm, vias 13 -> 1
- net Net-(D23-DIN): track 107.5 -> 8.17 mm, vias 11 -> 1
- net /Row 3: track 125.5 -> 32.0 mm, vias 15 -> 1
- net /Col 1: track 137.4 -> 46.1 mm, vias 8 -> 4
- net Net-(D40-DOUT): track 88.2 -> 16.5 mm, vias 7 -> 2
- net /Row 2: track 103.0 -> 31.4 mm, vias 13 -> 1
- net Net-(D13-A): track 81.7 -> 20.3 mm, vias 2 -> 1
- net /TX: track 69.6 -> 17.5 mm, vias 1 -> 0
- net Net-(D22-A): track 72.4 -> 20.5 mm, vias 6 -> 1
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- added copper zone on B.Cu, net GND
- removed copper zone on B.Cu, net (none)
- removed copper zone on F.Cu, net GND
Other:
- board size 150.7 x 99.3 mm -> 4.6 x 4.4 mm

Commit message: more routing
Parts:
- moved D1 0.41 mm to (159.6, 46.0)
- moved D2 0.41 mm to (162.5, 46.0)
- moved D3 0.41 mm to (165.3, 46.0)
Routing:
- net +5V: track 0.00 -> 315.0 mm, vias 0 -> 21
- net /Col 6: track 38.8 -> 232.8 mm, vias 4 -> 16
- net /Col 4: track 46.7 -> 232.1 mm, vias 4 -> 15
- net /Col 5: track 38.6 -> 204.5 mm, vias 3 -> 13
- net /Col 3: track 46.1 -> 206.6 mm, vias 4 -> 14
- net /Col 2: track 46.5 -> 201.2 mm, vias 4 -> 13
- net /Col 1: track 46.1 -> 158.4 mm, vias 4 -> 11
- net /Row 1: track 29.1 -> 124.7 mm, vias 1 -> 5
- net /Row 3: track 32.0 -> 119.1 mm, vias 1 -> 18
- net /Row 2: track 31.4 -> 97.3 mm, vias 1 -> 13
- net Net-(D12-A): track 20.3 -> 81.1 mm, vias 1 -> 4
- net Net-(D13-A): track 20.3 -> 63.0 mm, vias 1 -> 4
- net GND: track 0.00 -> 35.3 mm, vias 0 -> 27
- net Net-(D3-A): track 20.3 -> 55.5 mm, vias 1 -> 3
- net Net-(D11-A): track 20.3 -> 53.6 mm, vias 1 -> 4
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